File: Funkhaus-295/Funkhaus-295.kicad_sch (KiCad schematic)
At the start: 94 parts, among them SW1 SW_DPDT_x2, SW2 SW_Rotary3x4, SW3 SW_Rotary2x6, U1 TL074, U2 TL074, U3 TL074

Commit message: removed redundant 4M7 resistors
Parts:
- removed R33, R34, R35: 4M7, Resistor_THT:R_Axial_DIN0207_L6.3mm_D2.5mm_P2.54mm_Vertical, symbol Device:R
- renumbered R36 to R33, R37 to R34, R38 to R35, R39 to R36, R40 to R37, R41 to R38, R42 to R39, R43 to R40
Connections:
- net at R6.1, SW1.3 (C), SW1.4 (A): now also R32.2
- net at RV1.1, SW1.2 (B): no longer R32.2
Other:
- moved on the sheet: R32

Commit message: fixed RV1 wiring
Connections:
- net at C32.1, R4.1, RV1.3: no longer C2.1, RV1.2
- new net: C2.1, RV1.2
Other:
- note added: "R32-R40 can be soldered directly across the terminals of the switches"
- moved on the sheet: C1, C2, C3, R3, RV3

Commit message: update footprints, started pcb
Parts:
- C1, C10, C11, C12, C13, C14, C15, C16, C17, C18, C19, C2, C20, C21, C22, C23, C24, C25, C26, C27, C3, C4, C5, C6, C7, C8, C9: footprint (none) -> Capacitor_THT:C_Rect_L10.0mm_W2.5mm_P7.50mm_MKS4
- C28, C29, C30, C31, C37, C38, C39, C40, C41, C42: footprint Capacitor_THT:C_Disc_D5.0mm_W2.5mm_P5.00mm -> Capacitor_SMD:C_1206_3216Metric
- C32: footprint Capacitor_THT:CP_Radial_D10.0mm_P5.00mm -> Capacitor_THT:CP_Radial_D8.0mm_P5.00mm
- C35, C36: footprint Capacitor_THT:CP_Radial_D10.0mm_P5.00mm -> Capacitor_THT:CP_Radial_D5.0mm_P2.50mm
- RV1, RV2, RV3: footprint Connector_PinHeader_2.54mm:PinHeader_1x03_P2.54mm_Horizontal -> Connector_PinHeader_2.54mm:PinHeader_1x03_P2.54mm_Vertical
- SW1: footprint Connector_PinHeader_2.54mm:PinHeader_2x03_P2.54mm_Horizontal -> Connector_PinHeader_2.54mm:PinHeader_2x03_P2.54mm_Vertical
- SW2: footprint Connector_PinHeader_2.54mm:PinHeader_1x05_P2.54mm_Horizontal -> Connector_PinHeader_2.54mm:PinHeader_1x05_P2.54mm_Vertical
- SW3: footprint Connector_PinHeader_2.54mm:PinHeader_1x07_P2.54mm_Horizontal -> Connector_PinHeader_2.54mm:PinHeader_1x07_P2.54mm_Vertical

Commit message: updated schematic for kicad 8.0
Parts:
- removed C37, C38, C39, C40, C41, C42: 100n, Capacitor_SMD:C_1206_3216Metric, symbol Device:C
- removed SW1: SW_DPDT_x2, Connector_PinHeader_2.54mm:PinHeader_2x03_P2.54mm_Vertical, symbol Switch:SW_DPDT_x2
- removed SW2: SW_Rotary3x4, Connector_PinHeader_2.54mm:PinHeader_1x05_P2.54mm_Vertical, symbol Switch:SW_Rotary3x4
- removed SW3: SW_Rotary2x6, Connector_PinHeader_2.54mm:PinHeader_1x07_P2.54mm_Vertical, symbol Switch:SW_Rotary2x6
- added C37, C38, C39, C40, C41, C42: 100n, Capacitor_SMD:C_0805_2012Metric, symbol Device:C_Small
- added J1, J2: AudioJack2, Connector_PinHeader_2.54mm:PinHeader_1x02_P2.54mm_Vertical, symbol Connector_Audio:AudioJack2
- added SW1: SW_Rotary_3x4, Connector_PinHeader_2.54mm:PinHeader_1x05_P2.54mm_Vertical, symbol Switch:SW_Rotary_3x4
- added SW2: SW_Rotary_2x6, Connector_PinHeader_2.54mm:PinHeader_1x07_P2.54mm_Vertical, symbol Switch:SW_Rotary_2x6
- added SW4: SW_DPDT_x2, Connector_PinHeader_2.54mm:PinHeader_2x03_P2.54mm_Vertical, symbol Switch:SW_DPDT_x2
- C28, C29, C30, C31: footprint Capacitor_SMD:C_1206_3216Metric -> Capacitor_SMD:C_0805_2012Metric
- U1, U2, U3: footprint Package_DIP:DIP-14_W10.16mm -> Package_SO:SOIC-14_3.9x8.7mm_P1.27mm
Connections:
- net +12V: now also C37.1, C39.1, C41.1
- net -12V: now also C38.2, C40.2, C42.2
- net at R2.2, R32.1: now also SW4.1 (A), SW4.6 (C)
- net at R32.2, R6.1: now also SW4.3 (C), SW4.4 (A)
- net at R21.1, R34.2, R35.1: now also SW1.3
- net at R20.2, R21.2, R22.2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: now also SW1.1, SW2.13
- net at C24.1, C27.1, R40.2: now also SW2.6
- net at R20.1, R33.2, R34.1: now also SW1.2
- net at R22.1, R35.2: now also SW1.4
- net at C14.1, R37.2, R38.1: now also SW2.3
- net at C16.1, C19.1, R38.2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: now also SW2.4
- net at C20.1, C23.1, R39.2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: now also SW2.5
- net at C9.1, R36.2, R37.1: now also SW2.2
- net at C4.1, C7.1, R36.1: now also SW2.1
- net at R5.2: now also SW4.5 (B)
- net at RV2.2: now also SW1.13
- net at RV1.1: now also SW4.2 (B)
- net GND renamed GNDA
- net GNDA: now also J1.S, J2.S; no longer C35.2, C36.1
- net IN: no longer names the net of C33.1
- net IN: now also J1.T
- net OUT: no longer names the net of R31.1
- net OUT: now also J2.T
- new net GNDREF: C35.2, C36.1, C37.2, C38.1, C39.2, C40.1, C41.2, C42.1
Other:
- note removed: "R32-R40 can be soldered directly across the terminals of the switches"
- company: Robert-André Vettel -> Greybox Audio
- moved on the sheet: C15, C26, C29, C31, C33, C34, C35, C36, R25, R28, R29, R30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
