File: SIAM-295b/ClassA/siemens/siemens.kicad_sch (KiCad schematic)
At the start: 113 parts, among them J1 Conn_01x04_Pin, J2 Conn_01x08_Pin, J3 Conn_01x02_Pin, J4 Conn_01x02_Pin, Q1 BC549, Q10 BD139, Q11 BD139, Q12 BC549, Q2 BD139, Q3 BD139, Q4 BC549, Q5 BC549, Q6 BD139, Q7 BD139, Q8 BC549, Q9 BC549, SW1 SW_Rotary_2x6, SW2 SW_DPDT_x2

Commit message: started pcb
Parts:
- J1: value Conn_01x04_Pin -> PWR_IN
- J3: value Conn_01x02_Pin -> AUDIO_IN
- J4: value Conn_01x02_Pin -> AUDIO_OUT
- RV18, RV29, RV31, RV4: footprint (none) -> Potentiometer_THT:Potentiometer_ACP_CA6-H2,5_Horizontal
- SW1: footprint Connector_PinHeader_2.54mm:PinHeader_1x06_P2.54mm_Vertical -> Connector_PinHeader_2.54mm:PinHeader_1x07_P2.54mm_Vertical
- TP1, TP2, TP3, TP4: footprint (none) -> TestPoint:TestPoint_THTPad_1.0x1.0mm_Drill0.5mm
Connections:
- net +24V: now also J2.1 (Pin_1)
- net GND: now also J2.8 (Pin_8); no longer J2.7 (Pin_7)
- net at C20.2: now also J2.7 (Pin_7); no longer J2.6 (Pin_6)
- net at C13.2, C23.1: now also J2.4 (Pin_4); no longer J2.3 (Pin_3)
- net at C7.2: now also J2.6 (Pin_6); no longer J2.5 (Pin_5)
- net at C11.1, C21.1: now also J2.2 (Pin_2); no longer J2.1 (Pin_1)
- net at C12.2, C22.1: now also J2.3 (Pin_3); no longer J2.2 (Pin_2)
- net at C14.2: now also J2.5 (Pin_5); no longer J2.4 (Pin_4)
Other:
- moved on the sheet: J2
Changed lines of the file:
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@@
 			)
 		)
-		(property "Footprint" ""
+		(property "Footprint" "Potentiometer_THT:Potentiometer_ACP_CA6-H2,5_Horizontal"
 			(at 184.15 125.73 0)
 			(effects
@@
 			)
 		)
-		(property "Footprint" ""
+		(property "Footprint" "Potentiometer_THT:Potentiometer_ACP_CA6-H2,5_Horizontal"
 			(at 355.6 109.22 0)
 			(effects
@@
 			)
 		)
-		(property "Value" "Conn_01x02_Pin"
+		(property "Value" "AUDIO_IN"
 			(at 15.875 76.2 0)
 			(effects
@@
 			)
 		)
-		(property "Footprint" ""
+		(property "Footprint" "TestPoint:TestPoint_THTPad_1.0x1.0mm_Drill0.5mm"
 			(at 359.41 135.89 0)
 			(effects
@@
 			)
 		)
-		(property "Footprint" ""
+		(property "Footprint" "TestPoint:TestPoint_THTPad_1.0x1.0mm_Drill0.5mm"
 			(at 184.15 119.38 0)
 			(effects
@@
 	(symbol
 		(lib_id "Connector:Conn_01x08_Pin")
-		(at 246.38 198.12 90)
+		(at 243.84 198.12 90)
 		(unit 1)
 		(exclude_from_sim yes)
@@
 		(fields_autoplaced yes)
 		(property "Reference" "J2"
-			(at 247.65 200.66 90)
+			(at 245.11 200.66 90)
 			(effects
 				(font
@@
 		)
 		(property "Value" "Conn_01x08_Pin"
-			(at 247.65 203.2 90)
+			(at 245.11 203.2 90)
 			(effects
 				(font
@@
 		)
 		(property "Footprint" "Connector_PinHeader_2.54mm:PinHeader_1x08_P2.54mm_Vertical"
-			(at 246.38 198.12 0)
+			(at 243.84 198.12 0)
 			(effects
 				(font
@@
 		)
 		(property "Datasheet" "~"
-			(at 246.38 198.12 0)
+			(at 243.84 198.12 0)
 			(effects
 				(font
@@
 		)
 		(property "Description" "Generic connector, single row, 01x08, script generated"
-			(at 246.38 198.12 0)
+			(at 243.84 198.12 0)
 			(effects
 				(font
@@
 			)
 		)
-		(property "Value" "Conn_01x04_Pin"
+		(property "Value" "PWR_IN"
 			(at 90.17 36.83 90)
 			(effects
@@
 			)
 		)
-		(property "Footprint" ""
+		(property "Footprint" "Potentiometer_THT:Potentiometer_ACP_CA6-H2,5_Horizontal"
 			(at 327.66 109.22 0)
 			(effects
@@
 			)
 		)
-		(property "Value" "Conn_01x02_Pin"
+		(property "Value" "AUDIO_OUT"
 			(at 404.495 106.68 0)
 			(effects
@@
 			)
 		)
-		(property "Footprint" ""
+		(property "Footprint" "TestPoint:TestPoint_THTPad_1.0x1.0mm_Drill0.5mm"
 			(at 393.7 46.99 0)
 			(effects
@@
 			)
 		)
-		(property "Footprint" ""
+		(property "Footprint" "TestPoint:TestPoint_THTPad_1.0x1.0mm_Drill0.5mm"
 			(at 369.57 109.22 0)
 			(effects
@@
 			)
 		)
-		(property "Footprint" ""
+		(property "Footprint" "Potentiometer_THT:Potentiometer_ACP_CA6-H2,5_Horizontal"
 			(at 290.83 115.57 0)
 			(effects
@@
 			)
 		)
-		(property "Footprint" "Connector_PinHeader_2.54mm:PinHeader_1x06_P2.54mm_Vertical"
+		(property "Footprint" "Connector_PinHeader_2.54mm:PinHeader_1x07_P2.54mm_Vertical"
 			(at 274.32 139.7 0)
 			(effects

Commit message: update pcb
switch transistors & resistors to smd
Parts:
- removed Q1, Q12, Q4, Q5, Q8, Q9: BC549, Package_TO_SOT_THT:TO-92_Inline, symbol Transistor_BJT:BC549
- removed Q10, Q11, Q2, Q3, Q6, Q7: BD139, Package_TO_SOT_THT:TO-126-3_Vertical, symbol Transistor_BJT:BD139
- added Q1, Q12, Q4, Q5, Q8, Q9: BC849, Package_TO_SOT_SMD:SOT-23, symbol Transistor_BJT:BC849
- added Q10, Q11, Q2, Q3, Q6, Q7: BCX56, Package_TO_SOT_SMD:SOT-89-3, symbol Transistor_BJT:BCX56
- C9: footprint Capacitor_THT:C_Disc_D4.7mm_W2.5mm_P5.00mm -> Capacitor_SMD:C_0805_2012Metric
- R1, R10, R100, R101, R11, R12, R13, R14, R15, R16, R17, R18, R19, R2, R20, R21, R22, R23, R25, R26, R27, R28, R3, R30, R32, R33, R34, R35, R36, R37, R4, R5, R50, R51, R52, R53, R54, R6, R7, R8, R9: footprint Resistor_THT:R_Axial_DIN0207_L6.3mm_D2.5mm_P7.62mm_Horizontal -> Resistor_SMD:R_1206_3216Metric_Pad1.30x1.75mm_HandSolder
- R24, R29, R31, R38, R39, R40: footprint Resistor_THT:R_Axial_DIN0204_L3.6mm_D1.6mm_P2.54mm_Vertical -> Resistor_SMD:R_1206_3216Metric_Pad1.30x1.75mm_HandSolder
Connections:
- net +24V: now also Q12.3 (C)
- net at C30.1: now also Q2.3 (E), Q3.2 (C)
- net at R32.2: now also Q10.1 (B), Q9.2 (E)
- net at C6.1, R13.1, R15.1: now also Q7.2 (C)
- net at R28.2, RV29.1, RV3.3: now also Q8.1 (B)
- net at R6.2: now also Q3.3 (E)
- net at C2.2, R21.1, R4.2: now also Q3.1 (B)
- net at C16.1, J4.1 (Pin_1), RV31.2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: now also Q10.3 (E), Q11.2 (C)
- net at R10.2: now also Q4.2 (E)
- net at R26.1: now also Q8.3 (C), Q9.1 (B)
- net at C3.1, R1.1, R5.2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: now also Q1.3 (C)
- net at C17.1, R33.1, R34.1: now also Q10.2 (C)
- net at C17.2, R34.2, R35.2: now also Q11.1 (B)
- net at C8.1, R12.2, R17.2: now also Q5.3 (C)
- net at C1.1, R1.2, R2.1: now also Q1.1 (B)
- net at C18.1, R37.2: now also Q12.1 (B)
- net at C9.1, R12.1: now also Q4.3 (C), Q5.1 (B)
- net at C26.2, C9.2, R8.2: now also Q4.1 (B)
- net at R25.1, R27.2: now also Q8.2 (E)
- net at C34.1, R51.2, R54.1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: now also Q6.2 (C), Q7.3 (E)
- net at R20.2, R23.2: now also Q12.2 (E), Q9.3 (C)
- net at R36.2: now also Q11.3 (E)
- net at C6.2, R13.2, R14.2: now also Q6.1 (B)
- net at C2.1, R3.2, R5.1: now also Q2.2 (C)
- net at R16.2: now also Q6.3 (E)
- new net: Q5.2 (E), Q7.1 (B)
- new net: Q1.2 (E), Q2.1 (B)

Commit message: update pcb
successfully routed all components
Parts:
- SW1: footprint Connector_PinHeader_2.54mm:PinHeader_1x07_P2.54mm_Vertical -> Connector_PinHeader_2.54mm:PinHeader_2x07_P2.54mm_Vertical
Changed lines of the file:
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@@
 			)
 		)
-		(property "Footprint" "Connector_PinHeader_2.54mm:PinHeader_1x07_P2.54mm_Vertical"
+		(property "Footprint" "Connector_PinHeader_2.54mm:PinHeader_2x07_P2.54mm_Vertical"
 			(at 274.32 139.7 0)
 			(effects
